Commit message: add licensed robotiq 85

File: public/geometries/DROID/panda.urdf (robot description, URDF)
Before this commit: robot panda, 26 links, 25 joints
Links:
- removed link left_inner_finger
- removed link left_inner_knuckle
- removed link left_outer_finger
- removed link left_outer_knuckle
- removed link right_inner_finger
- removed link right_inner_knuckle
- removed link right_outer_finger
- removed link right_outer_knuckle
- added link robotiq_85_adapter_link; collision mesh filename=../robotiq/robotiq_2f_c2_gripper_visualization/meshes/robot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; visual mesh filename=../robotiq/robotiq_2f_c2_gripper_visualization/meshes/robot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
- added link robotiq_85_left_finger_link; collision mesh filename=../robotiq/robotiq_2f_c2_gripper_visualization/meshes/robot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; visual mesh filename=../robotiq/robotiq_2f_c2_gripper_visualization/meshes/robot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
- added link robotiq_85_left_finger_tip_link; collision mesh filename=../robotiq/robotiq_2f_c2_gripper_visualization/meshes/robot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; visual mesh filename=../robotiq/robotiq_2f_c2_gripper_visualization/meshes/robot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
- added link robotiq_85_left_inner_knuckle_link; collision mesh filename=../robotiq/robotiq_2f_c2_gripper_visualization/meshes/robot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; visual mesh filename=../robotiq/robotiq_2f_c2_gripper_visualization/meshes/robot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
- added link robotiq_85_left_knuckle_link; collision mesh filename=../robotiq/robotiq_2f_c2_gripper_visualization/meshes/robot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; visual mesh filename=../robotiq/robotiq_2f_c2_gripper_visualization/meshes/robot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
- added link robotiq_85_right_finger_link; collision mesh filename=../robotiq/robotiq_2f_c2_gripper_visualization/meshes/robot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; visual mesh filename=../robotiq/robotiq_2f_c2_gripper_visualization/meshes/robot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
- added link robotiq_85_right_finger_tip_link; collision mesh filename=../robotiq/robotiq_2f_c2_gripper_visualization/meshes/robot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; visual mesh filename=../robotiq/robotiq_2f_c2_gripper_visualization/meshes/robot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
- added link robotiq_85_right_inner_knuckle_link; collision mesh filename=../robotiq/robotiq_2f_c2_gripper_visualization/meshes/robot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; visual mesh filename=../robotiq/robotiq_2f_c2_gripper_visualization/meshes/robot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
- added link robotiq_85_right_knuckle_link; collision mesh filename=../robotiq/robotiq_2f_c2_gripper_visualization/meshes/robot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; visual mesh filename=../robotiq/robotiq_2f_c2_gripper_visualization/meshes/robot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
- link robotiq_85_base_link: mass 0.30915 -> None; geometry collision mesh filename=../robotiq/robotiq_2f_c2_gripper_visualization/meshes/robot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; visual mesh filename=../robotiq/robotiq_2f_c2_gripper_visualization/meshes/robot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
Joints:
- removed joint finger_joint
- removed joint left_inner_finger_joint
- removed joint left_inner_knuckle_joint
- removed joint left_outer_finger_joint
- removed joint right_inner_finger_joint
- removed joint right_inner_knuckle_joint
- removed joint right_outer_finger_joint
- removed joint right_outer_knuckle_joint
- removed joint test_name
- added joint robotiq_85_base_joint: type fixed, parent robotiq_85_adapter_link, child robotiq_85_base_link, origin xyz=.0085 0 -.0041 rpy=0 0 0, axis 1 0 0
- added joint robotiq_85_left_finger_joint: type fixed, parent robotiq_85_left_knuckle_link, child robotiq_85_left_finger_link, origin xyz=0 .00508 .03134 rpy=3.1415 0 0, axis 1 0 0, limit lower=0 upper=1.5707 effort=1000 velocity=2.0
- added joint robotiq_85_left_finger_tip_joint: type revolute, parent robotiq_85_left_inner_knuckle_link, child robotiq_85_left_finger_tip_link, origin xyz=0 .04196 -.0388 rpy=0 0 0, axis 1 0 0, limit lower=0 upper=1.5707 effort=1000 velocity=2.0, mimic joint=robotiq_85_left_knuckle_joint multiplier=-1
- added joint robotiq_85_left_inner_knuckle_joint: type revolute, parent robotiq_85_base_link, child robotiq_85_left_inner_knuckle_link, origin xyz=.04843 .0127 0 rpy=1.5707 1.5707 0, axis 1 0 0, limit lower=0 upper=1.5707 effort=1000 velocity=2.0, mimic joint=robotiq_85_left_knuckle_joint offset=0
- added joint robotiq_85_left_knuckle_joint: type revolute, parent robotiq_85_base_link, child robotiq_85_left_knuckle_link, origin xyz=.04191 .0306 0 rpy=-1.5707 1.5707 0, axis 1 0 0, limit lower=0 upper=.8575 effort=1000 velocity=2.0
- added joint robotiq_85_right_finger_joint: type fixed, parent robotiq_85_right_knuckle_link, child robotiq_85_right_finger_link, origin xyz=0 .00508 .03134 rpy=3.1415 0 0, axis 1 0 0, limit lower=0 upper=1.5707 effort=1000 velocity=2.0
- added joint robotiq_85_right_finger_tip_joint: type revolute, parent robotiq_85_right_inner_knuckle_link, child robotiq_85_right_finger_tip_link, origin xyz=0 .04196 -.0388 rpy=0 0 0, axis 1 0 0, limit lower=0 upper=1.5707 effort=1000 velocity=2.0, mimic joint=robotiq_85_left_knuckle_joint multiplier=-1
- added joint robotiq_85_right_inner_knuckle_joint: type revolute, parent robotiq_85_base_link, child robotiq_85_right_inner_knuckle_link, origin xyz=.04843 -.0127 0 rpy=-1.5707 -1.5707 0, axis 1 0 0, limit lower=0 upper=1.5707 effort=1000 velocity=2.0, mimic joint=robotiq_85_left_knuckle_joint offset=0
- added joint robotiq_85_right_knuckle_joint: type revolute, parent robotiq_85_base_link, child robotiq_85_right_knuckle_link, origin xyz=.04191 -.0306 0 rpy=1.5707 -1.5707 0, axis 1 0 0, limit lower=0 upper=1.5707 effort=1000 velocity=2.0, mimic joint=robotiq_85_left_knuckle_joint multiplier=1
- joint panda_joint8: child panda_link8 -> robotiq_85_adapter_link; origin xyz=0 0 0.107 rpy=0 0 0 -> xyz=0 0 0.1 rpy=0 -1.5707963267948966 0

Commit message: add pandas

File: public/geometries/DROID/panda.urdf (robot description, URDF)
Before this commit: robot panda, 27 links, 25 joints
Links:
- removed link panda_link0_sc
- removed link panda_link1_sc
- removed link panda_link2_sc
- removed link panda_link3_sc
- removed link panda_link4_sc
- removed link panda_link5_sc
- removed link panda_link6_sc
- removed link panda_link7_sc
- link panda_link0: mass None -> 0.629769273993887
- link panda_link1: mass None -> 4.970684
- link panda_link2: mass None -> 0.646926
- link panda_link3: mass None -> 3.228604
- link panda_link4: mass None -> 3.587895
- link panda_link5: mass None -> 1.225946
- link panda_link6: mass None -> 1.666555
- link panda_link7: mass None -> 7.35522e-01
- link panda_link8: mass None -> 1e-10
Joints:
- removed joint panda_link0_sc_joint
- removed joint panda_link1_sc_joint
- removed joint panda_link2_sc_joint
- removed joint panda_link3_sc_joint
- removed joint panda_link4_sc_joint
- removed joint panda_link5_sc_joint
- removed joint panda_link6_sc_joint
- removed joint panda_link7_sc_joint
- joint panda_joint1: limit lower=-2.8973 upper=2.8973 effort=87.0 velocity=2.175 -> lower=-2.9671 upper=2.9671 effort=87 velocity=2.5
- joint panda_joint2: limit lower=-1.7628 upper=1.7628 effort=87.0 velocity=2.175 -> lower=-1.8326 upper=1.8326 effort=87 velocity=2.5; origin xyz=0 0 0 rpy=-1.5707963267948966 0 0 -> xyz=0 0 0 rpy=-1.57079632679 0 0
- joint panda_joint3: limit lower=-2.8973 upper=2.8973 effort=87.0 velocity=2.175 -> lower=-2.9671 upper=2.9671 effort=87 velocity=2.5; origin xyz=0 -0.316 0 rpy=1.5707963267948966 0 0 -> xyz=0 -0.316 0 rpy=1.57079632679 0 0
- joint panda_joint4: limit lower=-3.0718 upper=-0.0698 effort=87.0 velocity=2.175 -> lower=-3.1416 upper=-0.4 effort=87 velocity=2.5; origin xyz=0.0825 0 0 rpy=1.5707963267948966 0 0 -> xyz=0.0825 0 0 rpy=1.57079632679 0 0
- joint panda_joint5: limit lower=-2.8973 upper=2.8973 effort=12.0 velocity=2.61 -> lower=-2.9671 upper=2.9671 effort=12 velocity=3; origin xyz=-0.0825 0.384 0 rpy=-1.5707963267948966 0 0 -> xyz=-0.0825 0.384 0 rpy=-1.57079632679 0 0
- joint panda_joint6: limit lower=-0.0175 upper=3.7525 effort=12.0 velocity=2.61 -> lower=-0.0873 upper=3.8223 effort=12 velocity=3; origin xyz=0 0 0 rpy=1.5707963267948966 0 0 -> xyz=0 0 0 rpy=1.57079632679 0 0
- joint panda_joint7: limit lower=-2.8973 upper=2.8973 effort=12.0 velocity=2.61 -> lower=-2.9671 upper=2.9671 effort=12 velocity=3; origin xyz=0.088 0 0 rpy=1.5707963267948966 0 0 -> xyz=0.088 0 0 rpy=1.57079632679 0 0

Commit message: add pandas

File: public/geometries/DROID/panda.urdf (robot description, URDF)
Before this commit: robot panda, 19 links, 17 joints
Joints:
- joint panda_joint8: origin xyz=0 0 0.1 rpy=0 -1.5707963267948966 0 -> xyz=0 0 0.107 rpy=0 -1.5707963267948966 0
